Commit message: changed paths

File: world_model_description/urdf/tanne1.urdf (robot description, URDF)
Before this commit: robot tree1, 1 links, 0 joints
Links:
- link base_link: geometry collision mesh filename=package://world_model_description/meshes/tanne1.dae; visual mesh filename=package://world_model_description/meshes/tanne1.dae

File: world_model_description/urdf/tanne12.urdf (robot description, URDF)
Before this commit: robot tree1, 1 links, 0 joints
Links:
- link base_link: geometry collision mesh filename=package://world_model_description/meshes/tanne12.dae; visual mesh filename=package://world_model_description/meshes/tanne12.dae

File: world_model_description/urdf/tanne2.urdf (robot description, URDF)
Before this commit: robot tree1, 1 links, 0 joints
Links:
- link base_link: geometry collision mesh filename=package://world_model_description/meshes/tanne2.dae; visual mesh filename=package://world_model_description/meshes/tanne2.dae

File: world_model_description/urdf/tanne21.urdf (robot description, URDF)
Before this commit: robot tree1, 1 links, 0 joints
Links:
- link base_link: geometry collision mesh filename=package://world_model_description/meshes/tanne21.dae; visual mesh filename=package://world_model_description/meshes/tanne21.dae

File: world_model_description/urdf/victim.urdf (robot description, URDF)
Before this commit: robot victim, 1 links, 0 joints
Links:
- link base_link: geometry collision mesh filename=package://world_model_description/meshes/victim.dae; visual mesh filename=package://world_model_description/meshes/victim.dae
