Commit message: added urdf

File: world_model_description/urdf/sphere.urdf (robot description, URDF)
Before this commit: robot sphere, 1 links, 0 joints
Links:
- link body: geometry collision mesh filename=package://sherpa_spatial_relations/meshes/cone.dae; visual mesh filename=package://world_model_description/meshes/sphere.dae
