Commit message: added new files

File: agents_model_description/urdf/human.urdf (robot description, URDF)
Before this commit: robot /, 75 links, 74 joints
Links:
- link camera_link: geometry collision mesh filename=package://agents_model_description/meshes/human/hokuyo.dae; visual mesh filename=package://agents_model_description/meshes/human/hokuyo.dae
- link head_z: geometry collision mesh filename=package://agents_model_description/meshes/human/Head.dae.stl; visual mesh filename=package://agents_model_description/meshes/human/Head.dae
- link l3_z: geometry collision mesh filename=package://agents_model_description/meshes/human/Body2.dae.s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; visual mesh filename=package://agents_model_description/meshes/human/Body2.dae
- link l5_z: geometry collision mesh filename=package://agents_model_description/meshes/human/Body1.dae.s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; visual mesh filename=package://agents_model_description/meshes/human/Body1.dae
- link left_foot_z: geometry collision mesh filename=package://agents_model_description/meshes/human/FootLeft.da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; visual mesh filename=package://agents_model_description/meshes/human/FootLeft.dae
- link left_hand_z: geometry collision mesh filename=package://agents_model_description/meshes/human/HandLeft.da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; visual mesh filename=package://agents_model_description/meshes/human/HandLeft.dae
- link left_lower_arm_z: geometry collision mesh filename=package://agents_model_description/meshes/human/LowerArmLef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; visual mesh filename=package://agents_model_description/meshes/human/LowerArmLef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
- link left_lower_leg_z: geometry collision mesh filename=package://agents_model_description/meshes/human/LowerLegLef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; visual mesh filename=package://agents_model_description/meshes/human/LowerLegLef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
- link left_shoulder_z: geometry collision mesh filename=package://agents_model_description/meshes/human/ShoulderLef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; visual mesh filename=package://agents_model_description/meshes/human/ShoulderLef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
- link left_toe_z: geometry collision mesh filename=package://agents_model_description/meshes/human/ToeLeft.dae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; visual mesh filename=package://agents_model_description/meshes/human/ToeLeft.dae
- link left_upper_arm_z: geometry collision mesh filename=package://agents_model_description/meshes/human/UpperArmLef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; visual mesh filename=package://agents_model_description/meshes/human/UpperArmLef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
- link left_upper_leg_z: geometry collision mesh filename=package://agents_model_description/meshes/human/UpperLegLef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; visual mesh filename=package://agents_model_description/meshes/human/UpperLegLef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
- link neck_z: geometry collision mesh filename=package://agents_model_description/meshes/human/Neck.dae.stl; visual mesh filename=package://agents_model_description/meshes/human/Neck.dae
- link pelvis_z: geometry collision mesh filename=package://agents_model_description/meshes/human/Hips.dae.stl; visual mesh filename=package://agents_model_description/meshes/human/Hips.dae
- link right_foot_z: geometry collision mesh filename=package://agents_model_description/meshes/human/FootRight.d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; visual mesh filename=package://agents_model_description/meshes/human/FootRight.d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
- link right_hand_z: geometry collision mesh filename=package://agents_model_description/meshes/human/HandRight.d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; visual mesh filename=package://agents_model_description/meshes/human/HandRight.d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
- link right_lower_arm_z: geometry collision mesh filename=package://agents_model_description/meshes/human/LowerArmRig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; visual mesh filename=package://agents_model_description/meshes/human/LowerArmRig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
- link right_lower_leg_z: geometry collision mesh filename=package://agents_model_description/meshes/human/LowerLegRig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; visual mesh filename=package://agents_model_description/meshes/human/LowerLegRig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
- link right_shoulder_z: geometry collision mesh filename=package://agents_model_description/meshes/human/ShoulderRig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; visual mesh filename=package://agents_model_description/meshes/human/ShoulderRig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
- link right_toe_z: geometry collision mesh filename=package://agents_model_description/meshes/human/ToeRight.da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; visual mesh filename=package://agents_model_description/meshes/human/ToeRight.dae
- link right_upper_arm_z: geometry collision mesh filename=package://agents_model_description/meshes/human/UpperArmRig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; visual mesh filename=package://agents_model_description/meshes/human/UpperArmRig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
- link right_upper_leg_z: geometry collision mesh filename=package://agents_model_description/meshes/human/UpperLegRig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; visual mesh filename=package://agents_model_description/meshes/human/UpperLegRig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
- link t12_z: geometry collision mesh filename=package://agents_model_description/meshes/human/Body3.dae.s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; visual mesh filename=package://agents_model_description/meshes/human/Body3.dae
- link t8_z: geometry collision mesh filename=package://agents_model_description/meshes/human/Body4.dae; visual mesh filename=package://agents_model_description/meshes/human/Body4.dae

Commit message: deleted all the build-files

File: agents_model_description/urdf/human.urdf (robot description, URDF)
Before this commit: robot /, 75 links, 74 joints
Links:
- removed link camera_depth_frame
- removed link camera_depth_optical_frame
- removed link camera_link
- removed link camera_rgb_frame
- removed link camera_rgb_optical_frame
- added link laser00_frame, mass 0.270; collision mesh filename=package://hector_sensors_description/meshes/hokuyo_utm30lx/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; visual mesh filename=package://hector_sensors_description/meshes/hokuyo_utm30lx/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
Joints:
- removed joint camera_depth_joint
- removed joint camera_depth_optical_joint
- removed joint camera_joint
- removed joint camera_rgb_joint
- removed joint camera_rgb_optical_joint
- added joint laser00_joint: type fixed, parent right_hand_y, child laser00_frame, origin xyz=-0.01 0 0 rpy=0 0 1.5

Commit message: added human

File: agents_model_description/urdf/human.urdf (robot description, URDF)
Before this commit: robot /, 71 links, 70 joints
Links:
- link laser00_frame: geometry 

Commit message: added human.urdf

File: agents_model_description/urdf/human.urdf (robot description, URDF)
Before this commit: robot /, 71 links, 70 joints
Links:
- removed link laser00_frame
- added link camera_depth_frame
- added link camera_depth_optical_frame
- added link camera_link, mass 0.200; collision box size=0.035 0.185 0.025; visual mesh filename=package://hector_sensors_description/meshes/asus_camera/asu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
- added link camera_rgb_frame
- added link camera_rgb_optical_frame
Joints:
- removed joint laser00_joint
- added joint camera_depth_joint: type fixed, parent camera_link, child camera_depth_frame, origin xyz=0.0 0.049 0.0 rpy=0 0 0
- added joint camera_depth_optical_joint: type fixed, parent camera_depth_frame, child camera_depth_optical_frame, origin xyz=0 0 0 rpy=-1.57079632679 0.0 -1.57079632679
- added joint camera_joint: type fixed, parent head_y, child camera_link, origin xyz=0.1 0.0 -0.03 rpy=0 0.349065850399 0
- added joint camera_rgb_joint: type fixed, parent camera_link, child camera_rgb_frame, origin xyz=0.0 0.022 0.0 rpy=0 0 0
- added joint camera_rgb_optical_joint: type fixed, parent camera_rgb_frame, child camera_rgb_optical_frame, origin xyz=0 0 0 rpy=-1.57079632679 0.0 -1.57079632679

Commit message: added new human.urdf

File: agents_model_description/urdf/human.urdf (robot description, URDF)
Before this commit: robot /, 75 links, 74 joints
Links:
- removed link camera_depth_frame
- removed link camera_depth_optical_frame
- removed link camera_link
- removed link camera_rgb_frame
- removed link camera_rgb_optical_frame
- added link cam_depth_frame
- added link cam_depth_optical_frame
- added link cam_link; collision mesh filename=package://hector_sensors_description/meshes/kinect_camera/k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; visual mesh filename=package://hector_sensors_description/meshes/kinect_camera/k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
- added link cam_rgb_frame
- added link cam_rgb_optical_frame
Joints:
- removed joint camera_depth_joint
- removed joint camera_depth_optical_joint
- removed joint camera_joint
- removed joint camera_rgb_joint
- removed joint camera_rgb_optical_joint
- added joint cam_depth_joint: type fixed, parent cam_link, child cam_depth_frame, origin xyz=0.0 -0.02 0.0 rpy=0 0 0
- added joint cam_depth_optical_joint: type fixed, parent cam_depth_frame, child cam_depth_optical_frame, origin xyz=0 0 0 rpy=-1.57079632679 0.0 -1.57079632679
- added joint cam_joint: type fixed, parent head_y, child cam_link, origin xyz=0.05 0.0 -0.06 rpy=0 0 0
- added joint cam_rgb_joint: type fixed, parent cam_link, child cam_rgb_frame, origin xyz=0.0 -0.0125 0.0 rpy=0 0 0
- added joint cam_rgb_optical_joint: type fixed, parent cam_rgb_frame, child cam_rgb_optical_frame, origin xyz=0 0 0 rpy=-1.57079632679 0.0 -1.57079632679
